Commit message: P1: fix SDF link poses (SDF≠URDF joint semantics) + clearance 1cm + lidar above mast
H1: Add explicit <pose> to all 11 links in model frame (SDF semantics: link pose ≠
joint pose; URDF joint/origin places child link, SDF does not). Wheels, casters,
scan, mast, camera now spawn at correct world positions.

H2: Raise base_link z 0.12→0.13 (1cm ground clearance). URDF still 0.12 — noted,
not fixed this phase.

Lidar (base_scan) raised z=0.285→0.625 to clear fork_mast top (z≈0.560). Mast was
blocking 10% of scan rays, causing Nav2 collision_monitor to block forward motion.
URDF lidar joint origin updated 0.155→0.495 to match.

Reset all <joint><pose> to 0 0 0 0 0 0 (anchor at child link origin).

Gate results:
  G1.1: H1 confirmed — all links were at origin pre-fix
  G1.2a: link poses match design table post-fix
  G1.2: GT Δ=1.368m ∈ [1.2,1.8]; |odom Δ−GT Δ|=0.000m ≤ 0.15m
  G1.3: Nav2 SUCCEEDED in 10.7s, 0 recoveries; GT dist to (0,0)=0.158m ≤ 1.0m (xy_tol=0.80)
  G1.4: start_demo ✓ /odom(1s) + Nav2(0s) warm=7s

Co-Authored-By: Claude Sonnet 4.6 <noreply@anthropic.com>

File: colcon_ws/src/warehouse_nav/urdf/warehouse_forklift.urdf (robot description, URDF)
Before this commit: robot warehouse_forklift, 12 links, 11 joints
Joints:
- joint lidar_joint: origin xyz=0 0 0.155 rpy=0 0 0 -> xyz=0 0 0.495 rpy=0 0 0
